File: kicad/mx/morizon-mx.kicad_pcb (KiCad board)
At the start: 2 copper layers, 266 x 76 mm, 116 parts, among them SW1 SW_Push, SW10 SW_Push, SW11 SW_Push, SW12 SW_Push, SW13 SW_Push, SW14 SW_Push, SW15 SW_Push, SW16 SW_Push, SW17 SW_Push, SW18 SW_Push, SW19 SW_Push, SW2 SW_Push, SW20 SW_Push, SW21 SW_Push, SW22 SW_Push, SW23 SW_Push, SW24 SW_Push, SW25 SW_Push, SW26 SW_Push, SW27 SW_Push, SW28 SW_Push, SW29 SW_Push, SW3 SW_Push, SW30 SW_Push, SW31 SW_Push, SW32 SW_Push, SW33 SW_Push, SW34 SW_Push, SW35 SW_Push, SW36 SW_Push, SW37 SW_Push, SW38 SW_Push, SW39 SW_Push, SW4 SW_Push, SW40 SW_Push, SW41 SW_Push, SW42 SW_Push, SW43 SW_Push, SW44 SW_Push, SW45 SW_Push, SW46 SW_Push, SW47 SW_Push, SW48 SW_Push, SW49 SW_Push, SW5 SW_Push, SW50 SW_Push, SW51 SW_Push, SW52 SW_Push, SW6 SW_Push, SW7 SW_Push, SW8 SW_Push, SW9 SW_Push, U1 PRO-MICRO

Commit message: Implement Morizon MX
Parts:
- added D53: D, horizon-footprints:D_SOD-123, B.Cu at (24.5, 147.2)
- added D54: D, horizon-footprints:D_SOD-123, B.Cu at (43.5, 147.2)
- added D55: D, horizon-footprints:D_SOD-123, B.Cu at (62.5, 147.2)
- added D56: D, horizon-footprints:D_SOD-123, B.Cu at (81.5, 147.2)
- added D57: D, horizon-footprints:D_SOD-123, B.Cu at (100.5, 147.2)
- added D58: D, horizon-footprints:D_SOD-123, B.Cu at (119.5, 147.2)
- added D59: D, horizon-footprints:D_SOD-123, B.Cu at (138.5, 147.2)
- added D60: D, horizon-footprints:D_SOD-123, B.Cu at (157.5, 147.2)
- added D61: D, horizon-footprints:D_SOD-123, B.Cu at (176.5, 147.2)
- added D62: D, horizon-footprints:D_SOD-123, B.Cu at (195.5, 147.2)
- added D63: D, horizon-footprints:D_SOD-123, B.Cu at (214.5, 147.2)
- added D64: D, horizon-footprints:D_SOD-123, B.Cu at (233.5, 147.2)
- added D65: D, horizon-footprints:D_SOD-123, B.Cu at (252.5, 147.2)
- added D66: D, horizon-footprints:D_SOD-123, B.Cu at (271.5, 147.2)
- added H9: Hole_Pad, horizon-footprints:Mount_M2, F.Cu at (148.0, 133.0)
- added SW53: SW_Push, horizon-footprints:SW_MX, F.Cu at (24.5, 142.5)
- added SW54: SW_Push, horizon-footprints:SW_MX, F.Cu at (43.5, 142.5)
- added SW55: SW_Push, horizon-footprints:SW_MX, F.Cu at (62.5, 142.5)
- added SW56: SW_Push, horizon-footprints:SW_MX, F.Cu at (81.5, 142.5)
- added SW57: SW_Push, horizon-footprints:SW_MX, F.Cu at (100.5, 142.5)
- added SW58: SW_Push, horizon-footprints:SW_MX, F.Cu at (119.5, 142.5)
- added SW59: SW_Push, horizon-footprints:SW_MX, F.Cu at (138.5, 142.5)
- added SW60: SW_Push, horizon-footprints:SW_MX, F.Cu at (157.5, 142.5)
- added SW61: SW_Push, horizon-footprints:SW_MX, F.Cu at (176.5, 142.5)
- added SW62: SW_Push, horizon-footprints:SW_MX, F.Cu at (195.5, 142.5)
- added SW63: SW_Push, horizon-footprints:SW_MX, F.Cu at (214.5, 142.5)
- added SW64: SW_Push, horizon-footprints:SW_MX, F.Cu at (233.5, 142.5)
- added SW65: SW_Push, horizon-footprints:SW_MX, F.Cu at (252.5, 142.5)
- added SW66: SW_Push, horizon-footprints:SW_MX, F.Cu at (271.5, 142.5)
- LOGO1: footprint horizon-footprints:Logo_Horizon_Small -> horizon-footprints:Logo_Morizon_Small
- LOGO2: footprint horizon-footprints:Logo_Horizon_H -> horizon-footprints:Logo_Morizon_M
- moved BTN1 10.0 mm to (134.0, 76.0)
- moved D1 10.0 mm to (24.5, 71.2)
- moved D10 10.0 mm to (233.5, 71.2)
- moved D11 10.0 mm to (252.5, 71.2)
- moved D12 10.0 mm to (271.5, 71.2)
- moved D13 10.0 mm to (24.5, 90.2)
- moved D14 10.0 mm to (43.5, 90.2)
- moved D15 10.0 mm to (62.5, 90.2)
- moved D16 10.0 mm to (81.5, 90.2)
- moved D17 10.0 mm to (100.5, 90.2)
- moved D18 10.0 mm to (119.5, 90.2)
- moved D19 10.0 mm to (176.5, 90.2)
- moved D2 10.0 mm to (43.5, 71.2)
- moved D20 10.0 mm to (195.5, 90.2)
- moved D21 10.0 mm to (214.5, 90.2)
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Connections:
- D10 pad 1: ROW1 -> ROW6
- D11 pad 1: ROW1 -> ROW6
- D12 pad 1: ROW1 -> ROW6
- D19 pad 1: ROW2 -> ROW7
- D20 pad 1: ROW2 -> ROW7
- D21 pad 1: ROW2 -> ROW7
- D22 pad 1: ROW2 -> ROW7
- D23 pad 1: ROW2 -> ROW7
- D24 pad 1: ROW2 -> ROW7
- D32 pad 1: ROW3 -> ROW8
- D33 pad 1: ROW3 -> ROW8
- D34 pad 1: ROW3 -> ROW8
- D35 pad 1: ROW3 -> ROW8
- D36 pad 1: ROW3 -> ROW8
- D37 pad 1: ROW3 -> ROW8
- D38 pad 1: ROW3 -> ROW8
- D46 pad 1: ROW4 -> ROW9
- D47 pad 1: ROW4 -> ROW9
- D48 pad 1: ROW4 -> ROW9
- D49 pad 1: ROW4 -> ROW9
- D50 pad 1: ROW4 -> ROW9
- D51 pad 1: ROW4 -> ROW9
- D52 pad 1: ROW4 -> ROW9
- D7 pad 1: ROW1 -> ROW6
- D8 pad 1: ROW1 -> ROW6
- D9 pad 1: ROW1 -> ROW6
- SW10 pad 1: COL12 -> COL5
- SW11 pad 1: COL13 -> COL6
- SW12 pad 1: COL14 -> COL7
- SW19 pad 1: COL9 -> COL2
- SW20 pad 1: COL10 -> COL3
- SW21 pad 1: COL11 -> COL4
- SW22 pad 1: COL12 -> COL5
- SW23 pad 1: COL13 -> COL6
- SW24 pad 1: COL14 -> COL7
- SW32 pad 1: COL8 -> COL1
- SW33 pad 1: COL9 -> COL2
- SW34 pad 1: COL10 -> COL3
- SW35 pad 1: COL11 -> COL4
- SW36 pad 1: COL12 -> COL5
- SW37 pad 1: COL13 -> COL6
- SW38 pad 1: COL14 -> COL7
- SW46 pad 1: COL8 -> COL1
- SW47 pad 1: COL9 -> COL2
- SW48 pad 1: COL10 -> COL3
- SW49 pad 1: COL11 -> COL4
- SW50 pad 1: COL12 -> COL5
- SW51 pad 1: COL13 -> COL6
- SW52 pad 1: COL14 -> COL7
- SW7 pad 1: COL9 -> COL2
- SW8 pad 1: COL10 -> COL3
- SW9 pad 1: COL11 -> COL4
- U1 pad 10: COL10 -> ROW8
- U1 pad 11: COL9 -> ROW9
- U1 pad 12: COL8 -> ROW10
- U1 pad 20: ROW4 -> (no net)
- U1 pad 6: COL14 -> ROW4
- U1 pad 7: COL13 -> ROW5
- U1 pad 8: COL12 -> ROW6
- U1 pad 9: COL11 -> ROW7
Routing:
- net COL7: track 34.3 -> 262.0 mm
- net COL6: track 88.1 -> 297.6 mm, vias 0 -> 1
- net ROW5: track 0.00 -> 199.7 mm, vias 0 -> 1
- net COL5: track 108.2 -> 300.3 mm, vias 0 -> 1
- net COL14: track 185.1 -> 0.00 mm
- net ROW10: track 0.00 -> 183.4 mm, vias 0 -> 1
- net COL4: track 129.3 -> 304.2 mm, vias 0 -> 1
- net ROW9: track 0.00 -> 167.0 mm, vias 0 -> 1
- net COL13: track 163.9 -> 0.00 mm
- net COL3: track 150.4 -> 308.0 mm, vias 0 -> 1
- net ROW2: track 304.9 -> 154.1 mm
- net ROW4: track 334.0 -> 183.2 mm
- net ROW8: track 0.00 -> 150.5 mm, vias 0 -> 1
- net ROW3: track 315.0 -> 166.8 mm
- net COL12: track 142.8 -> 0.00 mm
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Other:
- board size 266 x 76 mm -> 266 x 95 mm
- board text added: "github.com/skarrmann/morizon"
- board text added: "rev1 | MX"
- board text removed: "github.com/skarrmann/horizon"
- board text removed: "rev2.2 | MX"

Commit message: Upgrade project files to KiCad 6
Routing:
- net COL4: track 304.2 -> 313.0 mm
- net COL6: track 297.6 -> 306.4 mm
- net COL5: track 300.3 -> 309.2 mm
- net COL3: track 308.0 -> 316.8 mm
- net COL2: track 311.9 -> 320.7 mm
- net COL7: track 262.0 -> 267.8 mm
- net COL1: track 286.5 -> 289.3 mm
- net ROW5: track 199.7 -> 200.7 mm
Other:
- net class Default removed
- net class Power removed
- board text added: "rev1.1 | MX"
- board text removed: "rev1 | MX"

Commit message: Upgrade project files to KiCad 7
Other:
- board text added: "rev1.2 | MX"
- board text removed: "rev1.1 | MX"
